File: PCB/Aerospark v0.0.sch (EAGLE design)
At the start: 15 parts, among them T1 2N3904

Commit message: PCB Version 1.0 - Final
Other:
- moved on the sheet: JP1
Changed lines of the file:
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@@
 </plain>
 <instances>
-<instance part="JP1" gate="JP1" x="0" y="20.32">
-<attribute name="OC_NEWARK" x="0" y="20.32" size="1.778" layer="96" display="off"/>
-<attribute name="MF" x="0" y="20.32" size="1.778" layer="96" display="off"/>
-<attribute name="MPN" x="0" y="20.32" size="1.778" layer="96" display="off"/>
+<instance part="JP1" gate="JP1" x="7.62" y="22.86">
+<attribute name="OC_NEWARK" x="7.62" y="22.86" size="1.778" layer="96" display="off"/>
+<attribute name="MF" x="7.62" y="22.86" size="1.778" layer="96" display="off"/>
+<attribute name="MPN" x="7.62" y="22.86" size="1.778" layer="96" display="off"/>
 </instance>
 <instance part="U$2" gate="G$1" x="101.6" y="25.4">
@@
 <instance part="GND4" gate="1" x="129.54" y="-5.08"/>
 <instance part="GND1" gate="1" x="73.66" y="25.4"/>
-<instance part="GND2" gate="1" x="-20.32" y="-7.62"/>
+<instance part="GND2" gate="1" x="-12.7" y="-5.08"/>
 <instance part="GND5" gate="1" x="73.66" y="45.72" rot="R180"/>
 <instance part="GND6" gate="1" x="152.4" y="73.66"/>
@@
 <pinref part="GND5" gate="1" pin="GND"/>
 <junction x="73.66" y="43.18"/>
+<junction x="73.66" y="40.64"/>
 </segment>
 <segment>
 <pinref part="JP1" gate="JP1" pin="GND@6"/>
-<wire x1="-15.24" y1="7.62" x2="-20.32" y2="7.62" width="0.1524" layer="91"/>
+<wire x1="-7.62" y1="10.16" x2="-12.7" y2="10.16" width="0.1524" layer="91"/>
 <pinref part="GND2" gate="1" pin="GND"/>
-<wire x1="-20.32" y1="7.62" x2="-20.32" y2="5.08" width="0.1524" layer="91"/>
+<wire x1="-12.7" y1="10.16" x2="-12.7" y2="7.62" width="0.1524" layer="91"/>
 <pinref part="JP1" gate="JP1" pin="GND@9"/>
-<wire x1="-20.32" y1="5.08" x2="-20.32" y2="2.54" width="0.1524" layer="91"/>
-<wire x1="-20.32" y1="2.54" x2="-20.32" y2="0" width="0.1524" layer="91"/>
-<wire x1="-20.32" y1="0" x2="-20.32" y2="-2.54" width="0.1524" layer="91"/>
-<wire x1="-20.32" y1="-2.54" x2="-20.32" y2="-5.08" width="0.1524" layer="91"/>
-<wire x1="-15.24" y1="5.08" x2="-20.32" y2="5.08" width="0.1524" layer="91"/>
+<wire x1="-12.7" y1="7.62" x2="-12.7" y2="5.08" width="0.1524" layer="91"/>
+<wire x1="-12.7" y1="5.08" x2="-12.7" y2="2.54" width="0.1524" layer="91"/>
+<wire x1="-12.7" y1="2.54" x2="-12.7" y2="0" width="0.1524" layer="91"/>
+<wire x1="-12.7" y1="0" x2="-12.7" y2="-2.54" width="0.1524" layer="91"/>
+<wire x1="-7.62" y1="7.62" x2="-12.7" y2="7.62" width="0.1524" layer="91"/>
 <pinref part="JP1" gate="JP1" pin="GND@14"/>
-<wire x1="-15.24" y1="2.54" x2="-20.32" y2="2.54" width="0.1524" layer="91"/>
+<wire x1="-7.62" y1="5.08" x2="-12.7" y2="5.08" width="0.1524" layer="91"/>
 <pinref part="JP1" gate="JP1" pin="GND@20"/>
-<wire x1="-15.24" y1="0" x2="-20.32" y2="0" width="0.1524" layer="91"/>
+<wire x1="-7.62" y1="2.54" x2="-12.7" y2="2.54" width="0.1524" layer="91"/>
 <pinref part="JP1" gate="JP1" pin="GND@25"/>
-<wire x1="-15.24" y1="-2.54" x2="-20.32" y2="-2.54" width="0.1524" layer="91"/>
-<junction x="-20.32" y="-2.54"/>
-<junction x="-20.32" y="0"/>
-<junction x="-20.32" y="2.54"/>
-<junction x="-20.32" y="5.08"/>
-<junction x="-20.32" y="7.62"/>
+<wire x1="-7.62" y1="0" x2="-12.7" y2="0" width="0.1524" layer="91"/>
+<junction x="-12.7" y="0"/>
+<junction x="-12.7" y="2.54"/>
+<junction x="-12.7" y="5.08"/>
+<junction x="-12.7" y="7.62"/>
+<junction x="-12.7" y="10.16"/>
 </segment>
 <segment>
@@
 <segment>
 <pinref part="JP1" gate="JP1" pin="RXI"/>
-<wire x1="15.24" y1="35.56" x2="17.78" y2="35.56" width="0.1524" layer="91"/>
-<label x="17.78" y="35.56" size="1.27" layer="95" xref="yes"/>
+<wire x1="22.86" y1="38.1" x2="25.4" y2="38.1" width="0.1524" layer="91"/>
+<label x="25.4" y="38.1" size="1.27" layer="95" xref="yes"/>
 </segment>
 <segment>
@@
 <segment>
 <pinref part="JP1" gate="JP1" pin="TXO"/>
-<wire x1="15.24" y1="38.1" x2="17.78" y2="38.1" width="0.1524" layer="91"/>
-<label x="17.78" y="38.1" size="1.27" layer="95" xref="yes"/>
+<wire x1="22.86" y1="40.64" x2="25.4" y2="40.64" width="0.1524" layer="91"/>
+<label x="25.4" y="40.64" size="1.27" layer="95" xref="yes"/>
 </segment>
 </net>
@@
 <segment>
 <pinref part="JP1" gate="JP1" pin="5V@2"/>
-<wire x1="-15.24" y1="45.72" x2="-17.78" y2="45.72" width="0.1524" layer="91"/>
-<label x="-17.78" y="45.72" size="1.27" layer="95" rot="R180" xref="yes"/>
+<wire x1="-7.62" y1="48.26" x2="-10.16" y2="48.26" width="0.1524" layer="91"/>
+<label x="-10.16" y="48.26" size="1.27" layer="95" rot="R180" xref="yes"/>
 </segment>
 <segment>
@@
 <wire x1="60.96" y1="78.74" x2="60.96" y2="81.28" width="0.1524" layer="91"/>
 <label x="60.96" y="81.28" size="1.27" layer="95" rot="R90" xref="yes"/>
+<junction x="60.96" y="78.74"/>
 </segment>
 </net>
@@
 <segment>
 <pinref part="JP1" gate="JP1" pin="GP4"/>
-<wire x1="15.24" y1="15.24" x2="17.78" y2="15.24" width="0.1524" layer="91"/>
-<label x="17.78" y="15.24" size="1.27" layer="95" xref="yes"/>
+<wire x1="22.86" y1="17.78" x2="25.4" y2="17.78" width="0.1524" layer="91"/>
+<label x="25.4" y="17.78" size="1.27" layer="95" xref="yes"/>
 </segment>
 <segment>
@@
 <segment>
 <pinref part="JP1" gate="JP1" pin="GP17"/>
-<wire x1="15.24" y1="12.7" x2="17.78" y2="12.7" width="0.1524" layer="91"/>
-<label x="17.78" y="12.7" size="1.27" layer="95" xref="yes"/>
+<wire x1="22.86" y1="15.24" x2="25.4" y2="15.24" width="0.1524" layer="91"/>
+<label x="25.4" y="15.24" size="1.27" layer="95" xref="yes"/>
 </segment>
 <segment>
@@
 <segment>
 <pinref part="JP1" gate="JP1" pin="GP22"/>
-<wire x1="15.24" y1="7.62" x2="17.78" y2="7.62" width="0.1524" layer="91"/>
-<label x="17.78" y="7.62" size="1.27" layer="95" xref="yes"/>
+<wire x1="22.86" y1="10.16" x2="25.4" y2="10.16" width="0.1524" layer="91"/>
+<label x="25.4" y="10.16" size="1.27" layer="95" xref="yes"/>
 </segment>
 <segment>
@@
 <segment>
 <pinref part="JP1" gate="JP1" pin="GP27"/>
-<wire x1="15.24" y1="-2.54" x2="17.78" y2="-2.54" width="0.1524" layer="91"/>
-<label x="17.78" y="-2.54" size="1.27" layer="95" xref="yes"/>
+<wire x1="22.86" y1="0" x2="25.4" y2="0" width="0.1524" layer="91"/>
+<label x="25.4" y="0" size="1.27" layer="95" xref="yes"/>
 </segment>
 <segment>
@@
 <segment>
 <pinref part="JP1" gate="JP1" pin="3.3V@1"/>
-<wire x1="-15.24" y1="40.64" x2="-17.78" y2="40.64" width="0.1524" layer="91"/>
-<label x="-17.78" y="40.64" size="1.27" layer="95" rot="R180" xref="yes"/>
-</segment>
-<segment>
+<wire x1="-7.62" y1="43.18" x2="-10.16" y2="43.18" width="0.1524" layer="91"/>
+<label x="-10.16" y="43.18" size="1.27" layer="95" rot="R180" xref="yes"/>
+</segment>
+<segment>

Commit message: Updated PCB to v1.1
Parts:
- U$3: value SARANTEL-SR1202 -> JDGA-REMQV-ANTENNA; device Ava:SARANTEL-SR1202 -> Ava:JDGA-REMQV-ANTENNA; MPN SL1204SB -> (none); OC_NEWARK 96T7520 -> (none)
- renumbered C2 to C1, U$1 to RELAY
Connections:
- net GND: no longer U$2.10_GND, U$3.GND2
- net LOG: now also JP1.MISO; no longer JP1.GP17
- net PWR: now also JP1.SCLK; no longer JP1.GP4
- net SBD: now also JP1.MOSI; no longer JP1.GP22
Changed lines of the file:
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@@
 <attribute name="OC_NEWARK" value="unknown"/>
-</part>
-<part name="U$3" library="Ava" deviceset="SARANTEL-SR1202" device="">
-<attribute name="MF" value=""/>
-<attribute name="MPN" value="SL1204SB"/>
-<attribute name="OC_NEWARK" value="96T7520"/>
 </part>
 <part name="T1" library="transistor" deviceset="2N3904" device="" value="">
@@
 <part name="GND1" library="supply1" deviceset="GND" device=""/>
 <part name="GND2" library="supply1" deviceset="GND" device=""/>
-<part name="GND5" library="supply1" deviceset="GND" device=""/>
 <part name="GND6" library="supply1" deviceset="GND" device=""/>
 <part name="GND7" library="supply1" deviceset="GND" device=""/>
 <part name="GND8" library="supply1" deviceset="GND" device=""/>
-<part name="U$1" library="SparkFun-Electromechanical" deviceset="RELAY" device="PTH3">
+<part name="RELAY" library="SparkFun-Electromechanical" deviceset="RELAY" device="PTH3" value="">
 <attribute name="MF" value=""/>
 <attribute name="MPN" value=""/>
@@
 <attribute name="OC_NEWARK" value="unknown"/>
 </part>
-<part name="C2" library="SparkFun-Capacitors" deviceset="CAP" device="0805" value="100 NF">
+<part name="C1" library="SparkFun-Capacitors" deviceset="CAP" device="0805" value="100 NF">
 <attribute name="MF" value=""/>
 <attribute name="MPN" value=""/>
@@
 <attribute name="OC_NEWARK" value="34C8662"/>
 </part>
+<part name="U$3" library="Ava" deviceset="JDGA-REMQV-ANTENNA" device=""/>
 </parts>
 <sheets>
@@
 <attribute name="MPN" x="101.6" y="25.4" size="1.778" layer="96" display="off"/>
 </instance>
-<instance part="U$3" gate="G$1" x="48.26" y="33.02">
-<attribute name="OC_NEWARK" x="48.26" y="33.02" size="1.778" layer="96" display="off"/>
-<attribute name="MF" x="48.26" y="33.02" size="1.778" layer="96" display="off"/>
-<attribute name="MPN" x="48.26" y="33.02" size="1.778" layer="96" display="off"/>
-</instance>
 <instance part="T1" gate="G1" x="55.88" y="60.96">
 <attribute name="OC_NEWARK" x="55.88" y="60.96" size="1.778" layer="96" display="off"/>
@@
 <instance part="GND1" gate="1" x="73.66" y="25.4"/>
 <instance part="GND2" gate="1" x="-12.7" y="-5.08"/>
-<instance part="GND5" gate="1" x="73.66" y="45.72" rot="R180"/>
 <instance part="GND6" gate="1" x="152.4" y="73.66"/>
 <instance part="GND7" gate="1" x="152.4" y="63.5"/>
 <instance part="GND8" gate="1" x="152.4" y="53.34"/>
-<instance part="U$1" gate="G$1" x="76.2" y="73.66">
+<instance part="RELAY" gate="G$1" x="76.2" y="73.66">
 <attribute name="OC_NEWARK" x="76.2" y="73.66" size="1.778" layer="96" display="off"/>
 <attribute name="MF" x="76.2" y="73.66" size="1.778" layer="96" display="off"/>
@@
 <attribute name="MPN" x="99.06" y="73.66" size="1.778" layer="96" display="off"/>
 </instance>
-<instance part="C2" gate="G$1" x="139.7" y="35.56" rot="R180">
+<instance part="C1" gate="G$1" x="139.7" y="35.56" rot="R180">
 <attribute name="OC_NEWARK" x="139.7" y="35.56" size="1.778" layer="96" display="off"/>
 <attribute name="MF" x="139.7" y="35.56" size="1.778" layer="96" display="off"/>
@@
 <attribute name="MPN" x="45.72" y="60.96" size="1.778" layer="96" display="off"/>
 </instance>
+<instance part="U$3" gate="G$1" x="50.8" y="35.56"/>
 </instances>
 <busses>
@@
 <net name="N$1" class="0">
 <segment>
+<pinref part="U$2" gate="G$1" pin="11_RF_IN"/>
+<wire x1="68.58" y1="35.56" x2="78.74" y2="35.56" width="0.1524" layer="91"/>
 <pinref part="U$3" gate="G$1" pin="FEED"/>
-<pinref part="U$2" gate="G$1" pin="11_RF_IN"/>
-<wire x1="63.5" y1="35.56" x2="78.74" y2="35.56" width="0.1524" layer="91"/>
 </segment>
 </net>
@@
 <pinref part="GND3" gate="1" pin="GND"/>
 <junction x="139.7" y="25.4"/>
-<pinref part="C2" gate="G$1" pin="1"/>
+<pinref part="C1" gate="G$1" pin="1"/>
 </segment>
 <segment>
@@
 <segment>
 <pinref part="U$2" gate="G$1" pin="12_GND"/>
-<pinref part="U$3" gate="G$1" pin="GND"/>
 <wire x1="78.74" y1="30.48" x2="73.66" y2="30.48" width="0.1524" layer="91"/>
-<wire x1="73.66" y1="30.48" x2="63.5" y2="30.48" width="0.1524" layer="91"/>
+<wire x1="73.66" y1="30.48" x2="68.58" y2="30.48" width="0.1524" layer="91"/>
 <wire x1="73.66" y1="30.48" x2="73.66" y2="27.94" width="0.1524" layer="91"/>
 <pinref part="GND1" gate="1" pin="GND"/>
 <junction x="73.66" y="30.48"/>
-</segment>
-<segment>
-<pinref part="U$3" gate="G$1" pin="GND2"/>
-<pinref part="U$2" gate="G$1" pin="10_GND"/>
-<wire x1="78.74" y1="40.64" x2="73.66" y2="40.64" width="0.1524" layer="91"/>
-<wire x1="73.66" y1="40.64" x2="63.5" y2="40.64" width="0.1524" layer="91"/>
-<wire x1="73.66" y1="40.64" x2="73.66" y2="43.18" width="0.1524" layer="91"/>
-<pinref part="GND5" gate="1" pin="GND"/>
-<junction x="73.66" y="43.18"/>
-<junction x="73.66" y="40.64"/>
+<pinref part="U$3" gate="G$1" pin="GND"/>
 </segment>
 <segment>
@@
 <wire x1="22.86" y1="38.1" x2="25.4" y2="38.1" width="0.1524" layer="91"/>
 <label x="25.4" y="38.1" size="1.27" layer="95" xref="yes"/>
+<wire x1="22.86" y1="38.1" x2="25.4" y2="38.1" width="0.1524" layer="91"/>
+<wire x1="22.86" y1="38.1" x2="25.4" y2="38.1" width="0.1524" layer="91"/>
+<label x="25.4" y="38.1" size="1.27" layer="95" xref="yes"/>
 </segment>
 <segment>
@@
 <pinref part="D4" gate="G$1" pin="C"/>
 <wire x1="60.96" y1="76.2" x2="60.96" y2="78.74" width="0.1524" layer="91"/>
-<pinref part="U$1" gate="G$1" pin="COIL1"/>
+<pinref part="RELAY" gate="G$1" pin="COIL1"/>
 <wire x1="60.96" y1="78.74" x2="66.04" y2="78.74" width="0.1524" layer="91"/>
 <wire x1="60.96" y1="78.74" x2="60.96" y2="81.28" width="0.1524" layer="91"/>
@@
 <net name="PWR" class="0">
 <segment>
-<pinref part="JP1" gate="JP1" pin="GP4"/>
-<wire x1="22.86" y1="17.78" x2="25.4" y2="17.78" width="0.1524" layer="91"/>
-<label x="25.4" y="17.78" size="1.27" layer="95" xref="yes"/>
-</segment>
-<segment>
 <wire x1="124.46" y1="78.74" x2="121.92" y2="78.74" width="0.1524" layer="91"/>
 <label x="121.92" y="78.74" size="1.27" layer="95" rot="R180" xref="yes"/>
 <pinref part="PWR" gate="G$1" pin="A"/>
 </segment>
+<segment>
+<pinref part="JP1" gate="JP1" pin="SCLK"/>
+<wire x1="22.86" y1="33.02" x2="25.4" y2="33.02" width="0.1524" layer="91"/>
+<label x="25.4" y="33.02" size="1.27" layer="95" xref="yes"/>
+</segment>
 </net>
 <net name="LOG" class="0">
-<segment>
-<pinref part="JP1" gate="JP1" pin="GP17"/>
-<wire x1="22.86" y1="15.24" x2="25.4" y2="15.24" width="0.1524" layer="91"/>
-<label x="25.4" y="15.24" size="1.27" layer="95" xref="yes"/>
-</segment>
 <segment>
 <wire x1="124.46" y1="68.58" x2="121.92" y2="68.58" width="0.1524" layer="91"/>
@@
 <pinref part="LOG" gate="G$1" pin="A"/>
 </segment>
+<segment>
+<pinref part="JP1" gate="JP1" pin="MISO"/>
+<wire x1="22.86" y1="30.48" x2="25.4" y2="30.48" width="0.1524" layer="91"/>
+<label x="25.4" y="30.48" size="1.27" layer="95" xref="yes"/>
+</segment>
 </net>
 <net name="SBD" class="0">
-<segment>
-<pinref part="JP1" gate="JP1" pin="GP22"/>
-<wire x1="22.86" y1="10.16" x2="25.4" y2="10.16" width="0.1524" layer="91"/>
-<label x="25.4" y="10.16" size="1.27" layer="95" xref="yes"/>
-</segment>
 <segment>
 <wire x1="124.46" y1="58.42" x2="121.92" y2="58.42" width="0.1524" layer="91"/>
@@
 <pinref part="SBD" gate="G$1" pin="A"/>
 </segment>
+<segment>
+<pinref part="JP1" gate="JP1" pin="MOSI"/>
+<wire x1="22.86" y1="27.94" x2="25.4" y2="27.94" width="0.1524" layer="91"/>
+<label x="25.4" y="27.94" size="1.27" layer="95" xref="yes"/>
+</segment>
 </net>
 <net name="IGNT" class="0">
@@
 <pinref part="T1" gate="G1" pin="C"/>
 <wire x1="58.42" y1="66.04" x2="58.42" y2="68.58" width="0.1524" layer="91"/>
-<pinref part="U$1" gate="G$1" pin="COIL2"/>
+<pinref part="RELAY" gate="G$1" pin="COIL2"/>
 <wire x1="58.42" y1="68.58" x2="60.96" y2="68.58" width="0.1524" layer="91"/>
 <wire x1="60.96" y1="68.58" x2="66.04" y2="68.58" width="0.1524" layer="91"/>
 <wire x1="60.96" y1="68.58" x2="60.96" y2="71.12" width="0.1524" layer="91"/>
 <pinref part="D4" gate="G$1" pin="A"/>
+<junction x="60.96" y="68.58"/>
 </segment>
 </net>
@@
 <wire x1="139.7" y1="40.64" x2="147.32" y2="40.64" width="0.1524" layer="91"/>
 <label x="147.32" y="40.64" size="1.27" layer="95" xref="yes"/>
-<pinref part="C2" gate="G$1" pin="2"/>
+<pinref part="C1" gate="G$1" pin="2"/>
 </segment>
 </net>
 <net name="N$2" class="0">
 <segment>
-<pinref part="U$1" gate="G$1" pin="NC"/>
+<pinref part="RELAY" gate="G$1" pin="NC"/>
 <wire x1="83.82" y1="78.74" x2="86.36" y2="78.74" width="0.1524" layer="91"/>
 <wire x1="86.36" y1="78.74" x2="86.36" y2="73.66" width="0.1524" layer="91"/>
@@
 <net name="N$7" class="0">
 <segment>
-<pinref part="U$1" gate="G$1" pin="NO"/>
+<pinref part="RELAY" gate="G$1" pin="NO"/>
 <wire x1="83.82" y1="68.58" x2="86.36" y2="68.58" width="0.1524" layer="91"/>
 <wire x1="86.36" y1="68.58" x2="86.36" y2="71.12" width="0.1524" layer="91"/>
